File: ModuCard-Backplane-Sixth-Sense/CanTerminators.kicad_sch (KiCad schematic)
At the start: 14 parts, among them SW1 SW_DIP_x02, SW2 SW_DIP_x02

Commit message: erc -fix1
Parts:
- added R21, R22, R23, R24: 100Ω, PCM_JLCPCB:R_0603, symbol PCM_JLCPCB-Resistors:0603,100Ω
- added SW3, SW4: SW_DIP_x02, Button_Switch_THT:SW_DIP_SPSTx02_Slide_9.78x7.26mm_W7.62mm_P2.54mm, symbol Switch:SW_DIP_x02
Connections:
- new net: R24.1, SW4.2
- new net: R21.2, SW3.1
- new net: R22.1, SW3.2
- new net: R23.2, SW4.1
- new net Strobe1.+: R21.1, R23.1
- new net Strobe1.-: SW3.4, SW4.4
- new net Strobe2.+: R22.2, R24.2
- new net Strobe2.-: SW3.3, SW4.3
