File: ModuCard-Backplane-Sixth-Sense/Connector.kicad_sch (KiCad schematic)
At the start: 1 part, among them J17 09031967921

Commit message: erc -fix1
Connections:
- net CAN1.+: no longer J17.b4
- net CAN1.-: no longer J17.b5
- net CAN2.+: no longer J17.b7
- net CAN2.-: no longer J17.b8
- new net Strobe1.+: J17.b4
- new net Strobe1.-: J17.b5
- new net Strobe2.+: J17.b7
- new net Strobe2.-: J17.b8
