File: ModuCard-Backplane-Sixth-Sense/Ext-Connector.kicad_sch (KiCad schematic)
At the start: 1 part, among them J2 09031967921

Commit message: erc -fix1
Parts:
- J2: footprint Connector_DIN:DIN41612_R_3x32_Female_Horizontal_THT -> Connector_DIN:DIN41612_R_3x32_Male_Horizontal_THT
Connections:
- net +12V: now also J2.a17 (a16), J2.a18 (a15), J2.b17 (b16), J2.b18 (b15), J2.c17 (c16), J2.c18 (c15); no longer J2.a15, J2.a16, J2.b15, J2.b16, J2.c15, J2.c16
- net CAN1.+: now also J2.a29 (a4), J2.c29 (c4); no longer J2.a4, J2.b4, J2.c4
- net CAN1.-: now also J2.a28 (a5), J2.c28 (c5); no longer J2.a5, J2.b5, J2.c5
- net CAN2.+: now also J2.a26 (a7), J2.c26 (c7); no longer J2.a7, J2.b7, J2.c7
- net CAN2.-: now also J2.a25 (a8), J2.c25 (c8); no longer J2.a8, J2.b8, J2.c8
- net GND: now also J2.a11 (a22), J2.a12 (a21), J2.a13 (a20), J2.a15 (a18), J2.a16 (a17), J2.a24 (a9), J2.a27 (a6), J2.a30 (a3), J2.b11 (b22), J2.b12 (b21), J2.b13 (b20), J2.b15 (b18), J2.b16 (b17), J2.b24 (b9), J2.b27 (b6), J2.b30 (b3), J2.c11 (c22), J2.c12 (c21), J2.c13 (c20), J2.c15 (c18), J2.c16 (c17), J2.c24 (c9), J2.c27 (c6), J2.c30 (c3); no longer J2.a17, J2.a18, J2.a20, J2.a21, J2.a22, J2.a3, J2.a6, J2.a9, J2.b17, J2.b18, J2.b20, J2.b21, J2.b22, J2.b3, J2.b6, J2.b9, J2.c17, J2.c18, J2.c20, J2.c21, J2.c22, J2.c3, J2.c6, J2.c9
- net GPIOC0: now also J2.b23 (b10); no longer J2.b10
- net GPIOC1: now also J2.b22 (b11); no longer J2.b11
- net GPIOC2: now also J2.b21 (b12); no longer J2.b12
- net GPIOC3: now also J2.b20 (b13); no longer J2.b13
- net GPIOL0: now also J2.a23 (a10); no longer J2.a10
- net GPIOL1: now also J2.a22 (a11); no longer J2.a11
- net GPIOL2: now also J2.a21 (a12); no longer J2.a12
- net GPIOL3: now also J2.a20 (a13); no longer J2.a13
- net GPIOR0: now also J2.c23 (c10); no longer J2.c10
- net GPIOR1: now also J2.c22 (c11); no longer J2.c11
- net GPIOR2: now also J2.c21 (c12); no longer J2.c12
- net GPIOR3: now also J2.c20 (c13); no longer J2.c13
- net Index: now also J2.b31 (b2); no longer J2.b2
- net USB.D+: now also J2.c31 (c2); no longer J2.c2
- net USB.D-: now also J2.a31 (a2); no longer J2.a2
- net Vbat: now also J2.a10 (a23), J2.a2 (a31), J2.a3 (a30), J2.a4 (a29), J2.a5 (a28), J2.a6 (a27), J2.a7 (a26), J2.a8 (a25), J2.a9 (a24), J2.b10 (b23), J2.b2 (b31), J2.b3 (b30), J2.b4 (b29), J2.b5 (b28), J2.b6 (b27), J2.b7 (b26), J2.b8 (b25), J2.b9 (b24), J2.c10 (c23), J2.c2 (c31), J2.c3 (c30), J2.c4 (c29), J2.c5 (c28), J2.c6 (c27), J2.c7 (c26), J2.c8 (c25), J2.c9 (c24); no longer J2.a23, J2.a24, J2.a25, J2.a26, J2.a27, J2.a28, J2.a29, J2.a30, J2.a31, J2.b23, J2.b24, J2.b25, J2.b26, J2.b27, J2.b28, J2.b29, J2.b30, J2.b31, J2.c23, J2.c24, J2.c25, J2.c26, J2.c27, J2.c28, J2.c29, J2.c30, J2.c31
- new net Strobe1.+: J2.b29 (b4)
- new net Strobe1.-: J2.b28 (b5)
- new net Strobe2.+: J2.b26 (b7)
- new net Strobe2.-: J2.b25 (b8)
