File: ModuCard-Backplane-Sixth-Sense/FE2.1.kicad_sch (KiCad schematic)
At the start: 45 parts, among them U4 FE2.1, X2 X322512MSB4SI

Commit message: erc -fix1
Parts:
- removed C28: 100nF, PCM_JLCPCB:C_0402, symbol PCM_JLCPCB-Capacitors:0402,100nF,(2)
- added C41: 10uF, PCM_JLCPCB:C_0603, symbol PCM_JLCPCB-Capacitors:0603,10uF
- added D10, D9: LED, LED_THT:LED_D3.0mm, symbol Device:LED
Connections:
- net VD33_O is gone; now on net VD33: U4.9 (VD33_O)
- net GND: now also C41.2
- net at D20.2, D21.1, D22.2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: now also D32.1, D33.2, D10.2 (A), D9.1 (K); no longer D32.2, D33.1
- net VDD5 renamed +5V
- net +5V: now also C41.1
- new net: D10.1 (K), D32.2, D33.1, D9.2 (A), R37.2
Other:
- moved on the sheet: R37
