File: ModuCard-Backplane-Sixth-Sense/FE2.1.kicad_sch (KiCad schematic)
At the start: 47 parts, among them U4 FE2.1, X2 X322512MSB4SI

Commit message: fixed drv
Connections:
- net DRV: now also D10.2 (A), D20.2, D21.1, D22.2, D23.1, D24.2, D25.1, D26.2, D27.1, D28.2, D29.1, D30.2, D31.1, D32.1, D33.2, D9.1 (K), R38.1; no longer D34.2, R38.2
- new net: D34.2, R38.2
Other:
- moved on the sheet: D34, R38
Changed lines of the file:
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@@
 	)
 	(junction
-		(at 265.43 127)
-		(diameter 0)
-		(color 0 0 0 0)
-	)
-	(junction
 		(at 66.04 118.11)
 		(diameter 0)
@@
 	)
 	(junction
+		(at 265.43 127)
+		(diameter 0)
+		(color 0 0 0 0)
+	)
+	(junction
 		(at 49.53 152.4)
 		(diameter 0)
@@
 	)
 	(junction
+		(at 265.43 137.16)
+		(diameter 0)
+		(color 0 0 0 0)
+	)
+	(junction
 		(at 254 55.88)
 		(diameter 0)
@@
 	)
 	(junction
-		(at 265.43 144.78)
-		(diameter 0)
-		(color 0 0 0 0)
-	)
-	(junction
 		(at 254 123.19)
 		(diameter 0)
@@
 	(wire
 		(pts
-			(xy 265.43 135.89) (xy 265.43 127)
+			(xy 265.43 139.7) (xy 265.43 137.16)
 		)
 		(stroke
@@
 	(wire
 		(pts
-			(xy 265.43 143.51) (xy 265.43 144.78)
+			(xy 265.43 147.32) (xy 265.43 148.59)
 		)
 		(stroke
@@
 	(wire
 		(pts
+			(xy 261.62 137.16) (xy 265.43 137.16)
+		)
+		(stroke
+			(width 0)
+			(type default)
+		)
+	)
+	(wire
+		(pts
 			(xy 58.42 152.4) (xy 58.42 154.94)
 		)
@@
 	(wire
 		(pts
-			(xy 265.43 152.4) (xy 265.43 156.21)
+			(xy 265.43 156.21) (xy 265.43 160.02)
 		)
 		(stroke
@@
 	(wire
 		(pts
+			(xy 265.43 137.16) (xy 265.43 127)
+		)
+		(stroke
+			(width 0)
+			(type default)
+		)
+	)
+	(wire
+		(pts
 			(xy 254 39.37) (xy 254 43.18)
 		)
@@
 	(wire
 		(pts
-			(xy 251.46 144.78) (xy 265.43 144.78)
-		)
-		(stroke
-			(width 0)
-			(type default)
-		)
-	)
-	(wire
-		(pts
 			(xy 35.56 52.07) (xy 38.1 52.07)
 		)
@@
 		)
 	)
-	(label "DRV"
-		(at 251.46 144.78 180)
-		(effects
-			(font
-				(size 1.27 1.27)
-			)
-			(justify right bottom)
-		)
-	)
 	(label "USB6.D+"
 		(at 177.8 139.7 0)
@@
 		)
 	)
+	(label "DRV"
+		(at 261.62 137.16 180)
+		(effects
+			(font
+				(size 1.27 1.27)
+			)
+			(justify right bottom)
+		)
+	)
 	(label "OVCJ1"
 		(at 125.73 45.72 90)
@@
 	(symbol
 		(lib_id "PCM_JLCPCB-Resistors:0402,330Ω")
-		(at 265.43 139.7 0)
+		(at 265.43 143.51 0)
 		(unit 1)
 		(body_style 1)
@@
 		(fields_autoplaced yes)
 		(property "Reference" "R38"
-			(at 267.97 139.6999 0)
+			(at 267.97 143.5099 0)
 			(show_name no)
 			(do_not_autoplace no)
@@
 		)
 		(property "Value" "330Ω"
-			(at 265.43 139.7 90)
+			(at 265.43 143.51 90)
 			(show_name no)
 			(do_not_autoplace yes)
@@
 		)
 		(property "Footprint" "PCM_JLCPCB:R_0402"
-			(at 263.652 139.7 90)
+			(at 263.652 143.51 90)
 			(hide yes)
 			(show_name no)
@@
 		)
 		(property "Datasheet" "https://www.lcsc.com/datasheet/lcsc_datasheet_2205311900_UNI-ROYAL-Uniroyal-Elec-0402WGF3300TCE_C25104.pdf"
-			(at 265.43 139.7 0)
+			(at 265.43 143.51 0)
 			(hide yes)
 			(show_name no)
@@
 		)
 		(property "Description" "62.5mW Thick Film Resistors 50V ±100ppm/°C ±1% 330Ω 0402 Chip Resistor - Surface Mount ROHS"
-			(at 265.43 139.7 0)
+			(at 265.43 143.51 0)
 			(hide yes)
 			(show_name no)
@@
 		)
 		(property "LCSC" "C25104"
-			(at 265.43 139.7 0)
+			(at 265.43 143.51 0)
 			(hide yes)
 			(show_name no)
@@
 		)
 		(property "Stock" "1159127"
-			(at 265.43 139.7 0)
+			(at 265.43 143.51 0)
 			(hide yes)
 			(show_name no)
@@
 		)
 		(property "Price" "0.004USD"
-			(at 265.43 139.7 0)
+			(at 265.43 143.51 0)
 			(hide yes)
 			(show_name no)
@@
 		)
 		(property "Process" "SMT"
-			(at 265.43 139.7 0)
+			(at 265.43 143.51 0)
 			(hide yes)
 			(show_name no)
@@
 		)
 		(property "Minimum Qty" "20"
-			(at 265.43 139.7 0)
+			(at 265.43 143.51 0)
 			(hide yes)
 			(show_name no)
@@
 		)
 		(property "Attrition Qty" "10"
-			(at 265.43 139.7 0)
+			(at 265.43 143.51 0)
 			(hide yes)
 			(show_name no)
@@
 		)
 		(property "Class" "Basic Component"
-			(at 265.43 139.7 0)
+			(at 265.43 143.51 0)
 			(hide yes)
 			(show_name no)
@@
 		)
 		(property "Category" "Resistors,Chip Resistor - Surface Mount"
-			(at 265.43 139.7 0)
+			(at 265.43 143.51 0)
 			(hide yes)
 			(show_name no)
@@
 		)
 		(property "Manufacturer" "UNI-ROYAL(Uniroyal Elec)"
-			(at 265.43 139.7 0)
+			(at 265.43 143.51 0)
 			(hide yes)
 			(show_name no)
@@
 		)
 		(property "Part" "0402WGF3300TCE"
-			(at 265.43 139.7 0)
+			(at 265.43 143.51 0)
 			(hide yes)
 			(show_name no)
@@
 		)
 		(property "Resistance" "330Ω"
-			(at 265.43 139.7 0)
+			(at 265.43 143.51 0)
 			(hide yes)
 			(show_name no)
@@
 		)
 		(property "Power(Watts)" "62.5mW"
-			(at 265.43 139.7 0)
+			(at 265.43 143.51 0)
 			(hide yes)
 			(show_name no)
@@
 		)
 		(property "Type" "Thick Film Resistors"
-			(at 265.43 139.7 0)
+			(at 265.43 143.51 0)
 			(hide yes)
 			(show_name no)
@@
 		)
 		(property "Overload Voltage (Max)" "50V"
-			(at 265.43 139.7 0)
+			(at 265.43 143.51 0)
 			(hide yes)
 			(show_name no)
@@
 		)
 		(property "Operating Temperature Range" "-55°C~+155°C"
-			(at 265.43 139.7 0)
+			(at 265.43 143.51 0)
 			(hide yes)
 			(show_name no)
@@
 		)
 		(property "Tolerance" "±1%"
-			(at 265.43 139.7 0)
+			(at 265.43 143.51 0)
 			(hide yes)
 			(show_name no)
@@
 		)
 		(property "Temperature Coefficient" "±100ppm/°C"
-			(at 265.43 139.7 0)
+			(at 265.43 143.51 0)
 			(hide yes)
 			(show_name no)
@@
 	(symbol
 		(lib_id "PCM_JLCPCB-Diodes:LED,0603,Red")
-		(at 265.43 148.59 0)
+		(at 265.43 152.4 0)
 		(unit 1)
 		(body_style 1)
@@
 		(fields_autoplaced yes)
 		(property "Reference" "D34"
-			(at 267.97 147.2246 0)
+			(at 267.97 151.0346 0)
 			(show_name no)
 			(do_not_autoplace no)
@@
 		)
 		(property "Value" "Red"
-			(at 267.97 149.7647 0)
+			(at 267.97 153.5747 0)
 			(show_name no)
 			(do_not_autoplace no)
@@
 		)
 		(property "Footprint" "PCM_JLCPCB:D_0603"
-			(at 263.652 148.59 90)
+			(at 263.652 152.4 90)
 			(hide yes)
 			(show_name no)
@@
 		)
 		(property "Datasheet" "https://www.lcsc.com/datasheet/lcsc_datasheet_1810231112_Hubei-KENTO-Elec-KT-0603R_C2286.pdf"
-			(at 265.43 148.59 0)
+			(at 265.43 152.4 0)
 			(hide yes)
 			(show_name no)
@@
 		)
 		(property "Description" "-40°C~+85°C Red 0603 LED Indication - Discrete ROHS"
-			(at 265.43 148.59 0)
+			(at 265.43 152.4 0)
 			(hide yes)
 			(show_name no)
@@
 		)
 		(property "LCSC" "C2286"
-			(at 265.43 148.59 0)
+			(at 265.43 152.4 0)
 			(hide yes)
 			(show_name no)
@@
 		)
 		(property "Stock" "5373336"
-			(at 265.43 148.59 0)
+			(at 265.43 152.4 0)
 			(hide yes)
 			(show_name no)
@@
 		)
 		(property "Price" "0.009USD"
-			(at 265.43 148.59 0)
+			(at 265.43 152.4 0)
 			(hide yes)
 			(show_name no)
@@
 		)
 		(property "Process" "SMT"
-			(at 265.43 148.59 0)
+			(at 265.43 152.4 0)
 			(hide yes)
 			(show_name no)
@@
 		)
 		(property "Minimum Qty" "20"
-			(at 265.43 148.59 0)
+			(at 265.43 152.4 0)
 			(hide yes)
 			(show_name no)
@@
 		)
 		(property "Attrition Qty" "10"
-			(at 265.43 148.59 0)
+			(at 265.43 152.4 0)
 			(hide yes)
 			(show_name no)
@@
 		)
 		(property "Class" "Basic Component"
-			(at 265.43 148.59 0)
+			(at 265.43 152.4 0)
 			(hide yes)
 			(show_name no)
@@
 		)
 		(property "Category" "Optocouplers & LEDs & Infrared,Light Emitting Diodes (LED)"
-			(at 265.43 148.59 0)
+			(at 265.43 152.4 0)
 			(hide yes)
 			(show_name no)
@@
 		)
 		(property "Manufacturer" "Hubei KENTO Elec"
-			(at 265.43 148.59 0)
+			(at 265.43 152.4 0)
 			(hide yes)
 			(show_name no)
@@
 		)
 		(property "Part" "KT-0603R"
-			(at 265.43 148.59 0)
+			(at 265.43 152.4 0)
 			(hide yes)
 			(show_name no)
@@
 	(symbol
 		(lib_id "power:GND")
-		(at 265.43 156.21 0)
+		(at 265.43 160.02 0)
 		(unit 1)
 		(body_style 1)
@@
 		(fields_autoplaced yes)
 		(property "Reference" "#PWR052"
-			(at 265.43 162.56 0)
+			(at 265.43 166.37 0)
 			(hide yes)
 			(show_name no)
@@
 		)
 		(property "Value" "GND"
-			(at 265.43 161.29 0)
+			(at 265.43 165.1 0)
 			(show_name no)
 			(do_not_autoplace no)
@@
 		)
 		(property "Footprint" ""
-			(at 265.43 156.21 0)
+			(at 265.43 160.02 0)
 			(hide yes)
 			(show_name no)
@@
 		)
 		(property "Datasheet" ""
-			(at 265.43 156.21 0)
+			(at 265.43 160.02 0)
 			(hide yes)
 			(show_name no)
@@
 		)
 		(property "Description" "Power symbol creates a global label with name \"GND\" , ground"
-			(at 265.43 156.21 0)
+			(at 265.43 160.02 0)
 			(hide yes)
 			(show_name no)

Commit message: fixed PLL not being connected to 1.8v
Connections:
- net VD_DLL is gone; now on net VD18: U4.21 (VD_DLL)
Changed lines of the file:
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@@
+		)
+	)
+	(label "VD18"
+		(at 138.43 115.57 270)
+		(effects
+			(font
+				(size 1.27 1.27)
+			)
+			(justify right bottom)
 		)
 	)
@@
 		)
 	)
-	(label "VD_DLL"
-		(at 138.43 115.57 270)
-		(effects
-			(font
-				(size 1.27 1.27)
-			)
-			(justify right bottom)
-		)
-	)

Commit message: fixed OVCJ[1] not having pullup to 3v3
Parts:
- added R2: 10kΩ, PCM_JLCPCB:R_0402, symbol PCM_JLCPCB-Resistors:0402,10kΩ
Connections:
- net OVCJ1: now also R2.2
- net VD33: now also R2.1
