File: ModuCard-Backplane-Sixth-Sense/ModuCard-Backplane-Sixth-Sense.kicad_pcb (KiCad board)
At the start: 4 copper layers, 153.9 x 128.7 mm, 131 parts, among them J1 09031967921, J16 09031967921, J17 09031967921, J18 09031967921, J19 09031967921, J2 09031967921, J20 09031967921, J21 09031967921, J6 Conn_01x02_Pin, SW5 SW_DIP_x03, SW6 SW_DIP_x03, U1 LM5007MM, U3 AMS1117, U4 FE2.1, U801 FSUSB42UMX, U802 FSUSB42UMX, X2 X322512MSB4SI

Commit message: final check pinout
Parts:
- added J7: Conn_01x02_Pin, Connector_AMASS:AMASS_XT60-F_1x02_P7.20mm_Vertical, B.Cu at (271.0, 166.7)
- added Q1: BC847C, PCM_JLCPCB:Q_SOT-23, B.Cu at (278.0, 98.5)
- moved R39 6.60 mm to (279.5, 105.5), turned to 0 degrees
Connections:
- net /Ext-Connector/Index renamed /Ext-Connector/Index2
- D2 pad 1: GND -> Net-(D3-K)
- D3 pad 1: GND -> Net-(D3-K)
- J1 pad B1: GND -> /Ext-conn-M/Index1
- J1 pad B2: /Ext-conn-M/Index -> /Index2
- J16 pad b1: GND -> /Index1
- J16 pad b2: /Port1/Index -> /Index2
- J17 pad b1: GND -> /Index1
- J17 pad b2: /Port2/Index -> /Index2
- J18 pad b1: GND -> /Index1
- J18 pad b2: /Port3/Index -> /Index2
- J19 pad b1: GND -> /Index1
- J19 pad b2: /Port4/Index -> /Index2
- J2 pad b32: GND -> /Index1
- J20 pad b1: GND -> /Index1
- J20 pad b2: /Port5/Index -> /Index2
- J21 pad b1: GND -> /Index1
- J21 pad b2: /Ext-conn-M/Index -> /Index2
- R20 pad 2: /Ext-conn-M/Index -> /Ext-conn-M/Index1
- R39 pad 1: /Ext-conn-M/Index -> +3V3
- R802 pad 1: /Ext-conn-M/Index -> /Ext-conn-M/Index1
- R805 pad 1: /Ext-conn-M/Index -> /Ext-conn-M/Index1
Routing:
- net /Index1: track 0.00 -> 150.1 mm
- net /Index2: track 0.00 -> 127.7 mm
- net /Ext-conn-M/Index: track 101.1 -> 0.00 mm
- net /Ext-conn-M/Index1: track 0.00 -> 58.1 mm, vias 0 -> 2
- net Net-(D3-K): track 0.00 -> 7.35 mm
- net +5V: track 364.9 -> 358.5 mm
- net /FE2.1/DRV: track 217.6 -> 212.4 mm
- net +3V3: track 262.1 -> 259.3 mm, vias 6 -> 7
- net Net-(D3-A): track 6.64 -> 4.26 mm
- net GND: track 70.5 -> 69.6 mm, vias 850 -> 986
- net Net-(R5-Pad1): track 4.69 -> 4.12 mm
- net Vbat: vias 401 -> 356
Other:
- board text removed: "12V"
