File: ModuCard-Backplane-Sixth-Sense/ModuCard-Backplane-Sixth-Sense.kicad_pcb (KiCad board)
At the start: 4 copper layers, 153.9 x 128.7 mm, 133 parts, among them J1 09031967921, J16 09031967921, J17 09031967921, J18 09031967921, J19 09031967921, J2 09031967921, J20 09031967921, J21 09031967921, J6 Conn_01x02_Pin, J7 Conn_01x02_Pin, Q1 BC847C, SW5 SW_DIP_x03, SW6 SW_DIP_x03, U1 LM5007MM, U3 AMS1117, U4 FE2.1, U801 FSUSB42UMX, U802 FSUSB42UMX, X2 X322512MSB4SI

Commit message: fin
Parts:
- J6: moved to B.Cu
Connections:
- J16 pad b1: /Index1 -> /Port1/Index1
- J17 pad b1: /Index1 -> /Port2/Index1
- J18 pad b1: /Index1 -> /Port3/Index1
- J19 pad b1: /Index1 -> /Port4/Index1
- J2 pad b31: /Ext-Connector/Index2 -> /Index2
- J2 pad b32: /Index1 -> /Ext-Connector/Index1
- J20 pad b1: /Index1 -> /Port5/Index1
- J21 pad b1: /Index1 -> /Port6/Index1
- R26 pad 1: /Ext-Connector/Index2 -> /Ext-Connector/Index1
Routing:
- net /Index1: track 150.1 -> 0.00 mm
- net /Index2: track 127.7 -> 147.3 mm
- net /Ext-Connector/Index2: track 5.74 -> 0.00 mm
- net /Ext-Connector/Index1: track 0.00 -> 5.33 mm
- net /Port1/Index1: track 0.00 -> 2.22 mm
- net Net-(D34-Pad2): track 9.33 -> 7.94 mm
- net GND: track 69.6 -> 69.0 mm, vias 986 -> 1193
Other:
- board text removed: "12v"
- board text removed: "GND"
- board text removed: "GPIO 0"
- board text removed: "GPIO 1"
- board text removed: "GPIO 3"
- board text removed: "GPIO 4"
- board text removed: "[CAN 1 H]"
- board text removed: "[CAN 1 L]"
- board text removed: "[CAN 2 H]"
- board text removed: "[CAN 2 L]"
- board text removed: "[USB+]"
- board text removed: "[USB-]"
