File: ModuCard-Backplane-Sixth-Sense/ModuCard-Backplane-Sixth-Sense.kicad_sch (KiCad schematic)
At the start: 13 parts, among them U3 AMS1117

Commit message: erc -fix1
Parts:
- removed C3, C5: 10uF, PCM_JLCPCB:C_0603, symbol PCM_JLCPCB-Capacitors:0603,10uF
- removed C4, C6: 100nF, PCM_JLCPCB:C_0603, symbol PCM_JLCPCB-Capacitors:0603,100nF
- removed D2: RED, Diode_SMD:D_0402_1005Metric, symbol Device:LED
- removed R2: 1K2, Resistor_SMD:R_0402_1005Metric, symbol Device:R
- removed U3: AMS1117, PCM_JLCPCB:SOT-223-3_L6.5-W3.4-P2.30-LS7.0-BR, symbol PCM_JLCPCB-Power:LDO, 3.3V, 1A
- added D11, D12, D13: LED, LED_THT:LED_D3.0mm, symbol Device:LED
- added D2: Red, PCM_JLCPCB:D_0603, symbol PCM_JLCPCB-Diodes:LED,0603,Red
- added D3: LED, LED_THT:LED_D3.0mm_Clear, symbol Device:LED
- added D8: RED, Diode_SMD:D_0402_1005Metric, symbol Device:LED
- added R18: 1K2, Resistor_SMD:R_0402_1005Metric, symbol Device:R
- added R39: 330Ω, PCM_JLCPCB:R_0402, symbol PCM_JLCPCB-Resistors:0402,330Ω
Connections:
- net Ext-Connector2/Index is gone; now on net Ext-Connector/Index: R26.1
- net +12V: now also R19.2
- net +3V3: no longer R19.2
- net GND: now also D11.1 (K), D12.1 (K), D13.1 (K), D2.1, D3.1 (K), D8.1 (K)
- net at D4.2 (A), R19.1: now also D11.2 (A)
- net Vbat: now reaches R1.1
- net at D1.2 (A), R1.2: now also D12.2 (A)
- new net: D13.2 (A), D8.2 (A), R18.2
- new net: D2.2, D3.2 (A), R39.2
- new net +5V: R18.1
- new net Ext-conn-M/Index: R39.1
- no-connect marks 5 -> 7
Other:
- removed sheet Ext-Connector2
- added sheet Ext-conn-M (Ext-conn-M.kicad_sch)
- added sheet VRM (VRM.kicad_sch)
- sheet Can Split Terminators ports: added Strobe1{+ -}, Strobe2{+ -}; removed none
- sheet Ext-Connector ports: added Strobe1{+ -}, Strobe2{+ -}; removed none
- sheet Port1 ports: added Strobe1{+ -}, Strobe2{+ -}; removed none
- sheet Port2 ports: added Strobe1{+ -}, Strobe2{+ -}; removed none
- sheet Port3 ports: added Strobe1{+ -}, Strobe2{+ -}; removed none
- sheet Port4 ports: added Strobe1{+ -}, Strobe2{+ -}; removed none
- sheet Port5 ports: added Strobe1{+ -}, Strobe2{+ -}; removed none
- sheet Port6 ports: added Strobe1{+ -}, Strobe2{+ -}; removed none
- note added: "SLAVE MODE"
- moved on the sheet: D1, D4, R1, R19, R25, R26
