File: ModuCard-Backplane-Sixth-Sense/Mounting holes.kicad_sch (KiCad schematic)
At the start: 0 parts

Commit message: erc -fix1
Parts:
- added H1, H10, H11, H12, H13, H14, H15, H16, H2, H3, H4, H5, H6, H7, H8, H9: MountingHole, MountingHole:MountingHole_2.7mm_M2.5_DIN965_Pad, symbol Mechanical:MountingHole_Pad
Connections:
- no-connect marks 0 -> 16
