File: ModuCard-Backplane-Sixth-Sense/VRM.kicad_sch (KiCad schematic)
At the start: 23 parts, among them J4 Screw_Terminal_01x01, J5 Screw_Terminal_01x01, J6 Conn_01x02_Pin, U1 LM5007MM, U3 AMS1117

Commit message: project overhaul
Parts:
- removed D7: SS510, PCM_JLCPCB:D_SMA, symbol PCM_JLCPCB-Diodes:Schottky,SS510

Commit message: final check pinout
Parts:
- removed J4, J5: Screw_Terminal_01x01, symbol Connector:Screw_Terminal_01x01
- added J7: Conn_01x02_Pin, Connector_AMASS:AMASS_XT60-F_1x02_P7.20mm_Vertical, symbol Connector:Conn_01x02_Pin
Connections:
- net GND: now also J7.1 (Pin_1)
- net Vbat: now also J7.2 (Pin_2)
